File: pnp/pcb/mobo/misc_input.sch (KiCad schematic (older format))
At the start: 30 parts, among them J18 R_LIMIT, J19 P_LIMIT, J20 C_LIMIT, J60 X_LIMIT, J61 Y_LIMIT, J62 Z_LIMIT, U10 2SMPP-03, U11 LM358, U12 2SMPP-03, U13 INA126, U6 LM358, U9 INA126

Commit message: - Fixing LED JLCPCB code to be a yellow LED as well as updating R14 to be 680R per Issue #99 - Updates to the schematic to include LCSC and JLC part numbers. - Updates to generate renders of the board as well as an HTML BOM with digikey links, and a JLCPCB BOM.
Parts:
- J18, J19, J20, J60, J61, J62: LCSC (none) -> C2316
- R19, R20, R22, R23, R24, R25, R28, R29, R30, R32, R34, R35: Digikey (none) -> RMCF0805FT10K0CT-ND; JLCPCB (none) -> C17414; LCSC (none) -> C115295; Mouser (none) -> 71-CRCW080510K0FKEAC
- R21, R26: Digikey (none) -> 1712-CPF-A-0805B25KECT-ND; JLCPCB (none) -> C63863; LCSC (none) -> C63863; Mouser (none) -> 279-CPF-A-0805B25KE
- R27, R36: Digikey (none) -> RMCF0805FT1K00CT-ND; JLCPCB (none) -> C17513; LCSC (none) -> C702836; Mouser (none) -> 71-CRCW08051K00FKEAC
- R31, R33: Digikey (none) -> RMCF0805FT18K0CT-ND; JLCPCB (none) -> C17506; LCSC (none) -> C139848; Mouser (none) -> 667-ERJ-6ENF1802V
- U11, U6: Digikey (none) -> LM358DR2GOSCT-ND; JLCPCB (none) -> C7950; LCSC (none) -> C7950; Mouser (none) -> 863-LM358DR2G
- U13, U9: Digikey (none) -> 296-41257-1-ND; JLCPCB (none) -> C97254; LCSC (none) -> C350540; Mouser (none) -> 595-INA126UA/2K5
Changed lines of the file:
@@
 F 2 "Connector_JST:JST_XH_B3B-XH-A_1x03_P2.50mm_Vertical" H 1750 1250 50  0001 C CNN
 F 3 "~" H 1750 1250 50  0001 C CNN
+F 4 "C2316" H 1750 1250 50  0001 C CNN "LCSC"
 	1    1750 1250
 	-1   0    0    1
@@
 F 2 "Connector_JST:JST_XH_B3B-XH-A_1x03_P2.50mm_Vertical" H 1750 1800 50  0001 C CNN
 F 3 "~" H 1750 1800 50  0001 C CNN
+F 4 "C2316" H 1750 1800 50  0001 C CNN "LCSC"
 	1    1750 1800
 	-1   0    0    1
@@
 F 2 "Connector_JST:JST_XH_B3B-XH-A_1x03_P2.50mm_Vertical" H 1750 2350 50  0001 C CNN
 F 3 "~" H 1750 2350 50  0001 C CNN
+F 4 "C2316" H 1750 2350 50  0001 C CNN "LCSC"
 	1    1750 2350
 	-1   0    0    1
@@
 F 2 "Connector_JST:JST_XH_B3B-XH-A_1x03_P2.50mm_Vertical" H 1750 2950 50  0001 C CNN
 F 3 "~" H 1750 2950 50  0001 C CNN
+F 4 "C2316" H 1750 2950 50  0001 C CNN "LCSC"
 	1    1750 2950
 	-1   0    0    1
@@
 F 2 "Connector_JST:JST_XH_B3B-XH-A_1x03_P2.50mm_Vertical" H 1750 3500 50  0001 C CNN
 F 3 "~" H 1750 3500 50  0001 C CNN
+F 4 "C2316" H 1750 3500 50  0001 C CNN "LCSC"
 	1    1750 3500
 	-1   0    0    1
@@
 F 2 "Connector_JST:JST_XH_B3B-XH-A_1x03_P2.50mm_Vertical" H 1750 4050 50  0001 C CNN
 F 3 "~" H 1750 4050 50  0001 C CNN
+F 4 "C2316" H 1750 4050 50  0001 C CNN "LCSC"
 	1    1750 4050
 	-1   0    0    1
@@
 F 2 "Resistor_SMD:R_0805_2012Metric_Pad1.15x1.40mm_HandSolder" H 5350 3000 50  0001 C CNN
 F 3 "~" H 5350 3000 50  0001 C CNN
+F 4 "RMCF0805FT18K0CT-ND" H 5350 3000 50  0001 C CNN "Digikey"
+F 5 "C139848" H 5350 3000 50  0001 C CNN "LCSC"
+F 6 "667-ERJ-6ENF1802V" H 5350 3000 50  0001 C CNN "Mouser"
+F 7 "C17506" H 5350 3000 50  0001 C CNN "JLCPCB"
 	1    5350 3000
 	1    0    0    -1
@@
 F 2 "Package_SO:SOP-8_3.9x4.9mm_P1.27mm" H 4250 3100 50  0001 C CNN
 F 3 "" H 4250 3100 50  0001 C CNN
+F 4 "LM358DR2GOSCT-ND" H 4250 3100 50  0001 C CNN "Digikey"
+F 5 "C7950" H 4250 3100 50  0001 C CNN "LCSC"
+F 6 "863-LM358DR2G" H 4250 3100 50  0001 C CNN "Mouser"
+F 7 "C7950" H 4250 3100 50  0001 C CNN "JLCPCB"
 	1    4250 3100
 	1    0    0    -1
@@
 F 3 "~" H 2950 3150 50  0001 C CNN
 F 4 "1%" V 2950 3150 50  0000 C CNN "Notes"
+F 5 "1712-CPF-A-0805B25KECT-ND" H 2950 3150 50  0001 C CNN "Digikey"
+F 6 "C63863" H 2950 3150 50  0001 C CNN "LCSC"
+F 7 "279-CPF-A-0805B25KE" H 2950 3150 50  0001 C CNN "Mouser"
+F 8 "C63863" H 2950 3150 50  0001 C CNN "JLCPCB"
 	1    2950 3150
 	-1   0    0    1
@@
 F 2 "Resistor_SMD:R_0805_2012Metric_Pad1.15x1.40mm_HandSolder" H 6500 1650 50  0001 C CNN
 F 3 "~" H 6500 1650 50  0001 C CNN
+F 4 "RMCF0805FT1K00CT-ND" H 6500 1650 50  0001 C CNN "Digikey"
+F 5 "C702836" H 6500 1650 50  0001 C CNN "LCSC"
+F 6 "71-CRCW08051K00FKEAC" H 6500 1650 50  0001 C CNN "Mouser"
+F 7 "C17513" H 6500 1650 50  0001 C CNN "JLCPCB"
 	1    6500 1650
 	0    1    1    0
@@
 F 2 "Resistor_SMD:R_0805_2012Metric_Pad1.15x1.40mm_HandSolder" H 5350 3550 50  0001 C CNN
 F 3 "~" H 5350 3550 50  0001 C CNN
+F 4 "RMCF0805FT10K0CT-ND" H 5350 3550 50  0001 C CNN "Digikey"
+F 5 "C115295" H 5350 3550 50  0001 C CNN "LCSC"
+F 6 "71-CRCW080510K0FKEAC" H 5350 3550 50  0001 C CNN "Mouser"
+F 7 "C17414" H 5350 3550 50  0001 C CNN "JLCPCB"
 	1    5350 3550
 	1    0    0    -1
@@
 F 2 "Resistor_SMD:R_0805_2012Metric_Pad1.15x1.40mm_HandSolder" H 5650 3000 50  0001 C CNN
 F 3 "~" H 5650 3000 50  0001 C CNN
+F 4 "RMCF0805FT10K0CT-ND" H 5650 3000 50  0001 C CNN "Digikey"
+F 5 "C115295" H 5650 3000 50  0001 C CNN "LCSC"
+F 6 "71-CRCW080510K0FKEAC" H 5650 3000 50  0001 C CNN "Mouser"
+F 7 "C17414" H 5650 3000 50  0001 C CNN "JLCPCB"
 	1    5650 3000
 	1    0    0    -1
@@
 F 2 "Resistor_SMD:R_0805_2012Metric_Pad1.15x1.40mm_HandSolder" H 5650 3550 50  0001 C CNN
 F 3 "~" H 5650 3550 50  0001 C CNN
+F 4 "RMCF0805FT10K0CT-ND" H 5650 3550 50  0001 C CNN "Digikey"
+F 5 "C115295" H 5650 3550 50  0001 C CNN "LCSC"
+F 6 "71-CRCW080510K0FKEAC" H 5650 3550 50  0001 C CNN "Mouser"
+F 7 "C17414" H 5650 3550 50  0001 C CNN "JLCPCB"
 	1    5650 3550
 	1    0    0    -1
@@
 F 2 "Resistor_SMD:R_0805_2012Metric_Pad1.15x1.40mm_HandSolder" H 4950 3050 50  0001 C CNN
 F 3 "~" H 4950 3050 50  0001 C CNN
+F 4 "RMCF0805FT10K0CT-ND" H 4950 3050 50  0001 C CNN "Digikey"
+F 5 "C115295" H 4950 3050 50  0001 C CNN "LCSC"
+F 6 "71-CRCW080510K0FKEAC" H 4950 3050 50  0001 C CNN "Mouser"
+F 7 "C17414" H 4950 3050 50  0001 C CNN "JLCPCB"
 	1    4950 3050
 	0    1    1    0
@@
 F 2 "Resistor_SMD:R_0805_2012Metric_Pad1.15x1.40mm_HandSolder" H 3400 3400 50  0001 C CNN
 F 3 "~" H 3400 3400 50  0001 C CNN
+F 4 "RMCF0805FT10K0CT-ND" H 3400 3400 50  0001 C CNN "Digikey"
+F 5 "C115295" H 3400 3400 50  0001 C CNN "LCSC"
+F 6 "71-CRCW080510K0FKEAC" H 3400 3400 50  0001 C CNN "Mouser"
+F 7 "C17414" H 3400 3400 50  0001 C CNN "JLCPCB"
 	1    3400 3400
 	1    0    0    -1
@@
 F 2 "Resistor_SMD:R_0805_2012Metric_Pad1.15x1.40mm_HandSolder" H 3400 3000 50  0001 C CNN
 F 3 "~" H 3400 3000 50  0001 C CNN
+F 4 "RMCF0805FT10K0CT-ND" H 3400 3000 50  0001 C CNN "Digikey"
+F 5 "C115295" H 3400 3000 50  0001 C CNN "LCSC"
+F 6 "71-CRCW080510K0FKEAC" H 3400 3000 50  0001 C CNN "Mouser"
+F 7 "C17414" H 3400 3000 50  0001 C CNN "JLCPCB"
 	1    3400 3000
 	1    0    0    -1
@@
 F 2 "Package_SO:SOIC-8-1EP_3.9x4.9mm_P1.27mm_EP2.29x3mm" H 6400 2200 50  0001 C CNN
 F 3 "" H 6400 2200 50  0001 C CNN
+F 4 "296-41257-1-ND" H 6400 2200 50  0001 C CNN "Digikey"
+F 5 "C350540" H 6400 2200 50  0001 C CNN "LCSC"
+F 6 "595-INA126UA/2K5" H 6400 2200 50  0001 C CNN "Mouser"
+F 7 "C97254" H 6400 2200 50  0001 C CNN "JLCPCB"
 	1    6400 2200
 	1    0    0    -1
@@
 F 2 "Resistor_SMD:R_0805_2012Metric_Pad1.15x1.40mm_HandSolder" H 8600 5200 50  0001 C CNN
 F 3 "~" H 8600 5200 50  0001 C CNN
+F 4 "RMCF0805FT18K0CT-ND" H 8600 5200 50  0001 C CNN "Digikey"
+F 5 "C139848" H 8600 5200 50  0001 C CNN "LCSC"
+F 6 "667-ERJ-6ENF1802V" H 8600 5200 50  0001 C CNN "Mouser"
+F 7 "C17506" H 8600 5200 50  0001 C CNN "JLCPCB"
 	1    8600 5200
 	1    0    0    -1
@@
 F 2 "Package_SO:SOP-8_3.9x4.9mm_P1.27mm" H 7500 5300 50  0001 C CNN
 F 3 "" H 7500 5300 50  0001 C CNN
+F 4 "LM358DR2GOSCT-ND" H 7500 5300 50  0001 C CNN "Digikey"
+F 5 "C7950" H 7500 5300 50  0001 C CNN "LCSC"
+F 6 "863-LM358DR2G" H 7500 5300 50  0001 C CNN "Mouser"
+F 7 "C7950" H 7500 5300 50  0001 C CNN "JLCPCB"
 	1    7500 5300
 	1    0    0    -1
@@
 F 3 "~" H 6200 5350 50  0001 C CNN
 F 4 "1%" V 6200 5350 50  0000 C CNN "Notes"
+F 5 "1712-CPF-A-0805B25KECT-ND" H 6200 5350 50  0001 C CNN "Digikey"
+F 6 "C63863" H 6200 5350 50  0001 C CNN "LCSC"
+F 7 "279-CPF-A-0805B25KE" H 6200 5350 50  0001 C CNN "Mouser"
+F 8 "C63863" H 6200 5350 50  0001 C CNN "JLCPCB"
 	1    6200 5350
 	-1   0    0    1
@@
 F 2 "Resistor_SMD:R_0805_2012Metric_Pad1.15x1.40mm_HandSolder" H 9750 3850 50  0001 C CNN
 F 3 "~" H 9750 3850 50  0001 C CNN
+F 4 "RMCF0805FT1K00CT-ND" H 9750 3850 50  0001 C CNN "Digikey"
+F 5 "C702836" H 9750 3850 50  0001 C CNN "LCSC"
+F 6 "71-CRCW08051K00FKEAC" H 9750 3850 50  0001 C CNN "Mouser"
+F 7 "C17513" H 9750 3850 50  0001 C CNN "JLCPCB"
 	1    9750 3850
 	0    1    1    0
@@
 F 2 "Resistor_SMD:R_0805_2012Metric_Pad1.15x1.40mm_HandSolder" H 8600 5750 50  0001 C CNN
 F 3 "~" H 8600 5750 50  0001 C CNN
+F 4 "RMCF0805FT10K0CT-ND" H 8600 5750 50  0001 C CNN "Digikey"
+F 5 "C115295" H 8600 5750 50  0001 C CNN "LCSC"
+F 6 "71-CRCW080510K0FKEAC" H 8600 5750 50  0001 C CNN "Mouser"
+F 7 "C17414" H 8600 5750 50  0001 C CNN "JLCPCB"
 	1    8600 5750
 	1    0    0    -1
@@
 F 2 "Resistor_SMD:R_0805_2012Metric_Pad1.15x1.40mm_HandSolder" H 8900 5200 50  0001 C CNN
 F 3 "~" H 8900 5200 50  0001 C CNN
+F 4 "RMCF0805FT10K0CT-ND" H 8900 5200 50  0001 C CNN "Digikey"
+F 5 "C115295" H 8900 5200 50  0001 C CNN "LCSC"
+F 6 "71-CRCW080510K0FKEAC" H 8900 5200 50  0001 C CNN "Mouser"
+F 7 "C17414" H 8900 5200 50  0001 C CNN "JLCPCB"
 	1    8900 5200
 	1    0    0    -1
@@
 F 2 "Resistor_SMD:R_0805_2012Metric_Pad1.15x1.40mm_HandSolder" H 8900 5750 50  0001 C CNN
 F 3 "~" H 8900 5750 50  0001 C CNN
+F 4 "RMCF0805FT10K0CT-ND" H 8900 5750 50  0001 C CNN "Digikey"
+F 5 "C115295" H 8900 5750 50  0001 C CNN "LCSC"
+F 6 "71-CRCW080510K0FKEAC" H 8900 5750 50  0001 C CNN "Mouser"
+F 7 "C17414" H 8900 5750 50  0001 C CNN "JLCPCB"
 	1    8900 5750
 	1    0    0    -1
@@
 F 2 "Resistor_SMD:R_0805_2012Metric_Pad1.15x1.40mm_HandSolder" H 8200 5250 50  0001 C CNN
 F 3 "~" H 8200 5250 50  0001 C CNN
+F 4 "RMCF0805FT10K0CT-ND" H 8200 5250 50  0001 C CNN "Digikey"
+F 5 "C115295" H 8200 5250 50  0001 C CNN "LCSC"
+F 6 "71-CRCW080510K0FKEAC" H 8200 5250 50  0001 C CNN "Mouser"
+F 7 "C17414" H 8200 5250 50  0001 C CNN "JLCPCB"
 	1    8200 5250
 	0    1    1    0
@@
 F 2 "Resistor_SMD:R_0805_2012Metric_Pad1.15x1.40mm_HandSolder" H 6650 5600 50  0001 C CNN
 F 3 "~" H 6650 5600 50  0001 C CNN
+F 4 "RMCF0805FT10K0CT-ND" H 6650 5600 50  0001 C CNN "Digikey"
+F 5 "C115295" H 6650 5600 50  0001 C CNN "LCSC"
+F 6 "71-CRCW080510K0FKEAC" H 6650 5600 50  0001 C CNN "Mouser"
+F 7 "C17414" H 6650 5600 50  0001 C CNN "JLCPCB"
 	1    6650 5600
 	1    0    0    -1
@@
 F 2 "Resistor_SMD:R_0805_2012Metric_Pad1.15x1.40mm_HandSolder" H 6650 5200 50  0001 C CNN
 F 3 "~" H 6650 5200 50  0001 C CNN
+F 4 "RMCF0805FT10K0CT-ND" H 6650 5200 50  0001 C CNN "Digikey"
+F 5 "C115295" H 6650 5200 50  0001 C CNN "LCSC"
+F 6 "71-CRCW080510K0FKEAC" H 6650 5200 50  0001 C CNN "Mouser"
+F 7 "C17414" H 6650 5200 50  0001 C CNN "JLCPCB"
 	1    6650 5200
 	1    0    0    -1
@@
 F 2 "Package_SO:SOIC-8-1EP_3.9x4.9mm_P1.27mm_EP2.29x3mm" H 9650 4400 50  0001 C CNN
 F 3 "" H 9650 4400 50  0001 C CNN
+F 4 "296-41257-1-ND" H 9650 4400 50  0001 C CNN "Digikey"
+F 5 "C350540" H 9650 4400 50  0001 C CNN "LCSC"
+F 6 "595-INA126UA/2K5" H 9650 4400 50  0001 C CNN "Mouser"
+F 7 "C97254" H 9650 4400 50  0001 C CNN "JLCPCB"
 	1    9650 4400
 	1    0    0    -1
