File: pnp/pcb/mobo/misc_output.sch (KiCad schematic (older format))
At the start: 43 parts, among them J10 MF3, J11 MF4, J12 DOWNWARDS_LIGHT, J13 UPWARDS_LIGHT, J14 5V_INJECTION, J16 RS-485_2, J17 RS-485_3, J21 AUX1, J22 AUX2, J23 QWIIC1, J24 QWIIC2, J25 RS-485_1, J6 SERVO1, J7 SERVO2, J8 MF1, J9 MF2, Q1 TSM900N06, Q2 TSM900N06, Q3 TSM900N06, Q4 TSM900N06, U2 SP3485EN, U3 SP3485EN, U4 SP3485EN

Commit message: - Fixing LED JLCPCB code to be a yellow LED as well as updating R14 to be 680R per Issue #99 - Updates to the schematic to include LCSC and JLC part numbers. - Updates to generate renders of the board as well as an HTML BOM with digikey links, and a JLCPCB BOM.
Parts:
- C26, C27, C28: Digikey (none) -> 1276-1180-1-ND; JLCPCB (none) -> C49678; LCSC (none) -> C360619; Mouser (none) -> 581-08055C104K
- D3: Digikey (none) -> 732-4987-1-ND; JLCPCB (none) -> C2296; LCSC (none) -> C779458; Mouser (none) -> 710-150080YS75000
- D6, D7, D8, D9: JLCPCB (none) -> C64898; LCSC (none) -> C64898
- J10, J11, J14, J8, J9: LCSC (none) -> C20079
- J12, J13, J6, J7: LCSC (none) -> C2316
- J16, J17: LCSC (none) -> C37815
- J21, J22: LCSC (none) -> C5665
- J23, J24: LCSC (none) -> C145961
- J25: LCSC (none) -> C601936
- Q1, Q2, Q3, Q4: LCSC (none) -> C396085
- R10, R11, R12: Digikey (none) -> A129741CT-ND; JLCPCB (none) -> C17557; LCSC (none) -> C104115; Mouser (none) -> 667-ERJ-6ENF2200V
- R2, R3, R4, R5: JLCPCB (none) -> C17798; LCSC (none) -> C139848
- R37: Digikey (none) -> A126343CT-ND; JLCPCB (none) -> C25270; LCSC (none) -> C294691; Mouser (none) -> 71-CRCW0805180RFKEA
- R6, R7, R8, R9: JLCPCB (none) -> C17407; LCSC (none) -> C702859
- U2, U3, U4: Digikey (none) -> 1016-1817-1-ND; JLCPCB (none) -> C8963; LCSC (none) -> C19738; Mouser (none) -> 701-SP3485EN-L
