File: pnp/pcb/mobo/motor_control.sch (KiCad schematic (older format))
At the start: 49 parts, among them J1 X_MOTOR, J2 Y_MOTOR1, J3 Z_MOTOR, J37 P_MOTOR, J38 C_MOTOR, J4 R_MOTOR, J48 Y_MOTOR2

Commit message: - Fixing LED JLCPCB code to be a yellow LED as well as updating R14 to be 680R per Issue #99 - Updates to the schematic to include LCSC and JLC part numbers. - Updates to generate renders of the board as well as an HTML BOM with digikey links, and a JLCPCB BOM.
Parts:
- C1, C2, C3, C4, C5, C6: Digikey (none) -> 493-2203-1-ND; JLCPCB (none) -> C99837; LCSC (none) -> C263958; Mouser (none) -> 647-UWT1V101MCL1S
- J1, J2, J3, J37, J38, J4, J48: LCSC (none) -> C37815
- JP1, JP10, JP11, JP12, JP13, JP14, JP15, JP16, JP17, JP18, JP19, JP2, JP20, JP21, JP22, JP23, JP24, JP3, JP4, JP5, JP6, JP7, JP8, JP9: LCSC (none) -> C2337
- R43, R44, R45, R46, R47, R48: Digikey (none) -> RMCF0805FT1K00CT-ND; JLCPCB (none) -> C17513; LCSC (none) -> C702836; Mouser (none) -> 71-CRCW08051K00FKEAC
